Commit message: add minor fixes in wheels length, friction values and added plugins for drive and laser scan

File: my_rb1_description/urdf/my_rb1_robot.urdf (robot description, URDF)
Before this commit: robot rb1_robot, 7 links, 6 joints
Links:
- link left_wheel: geometry collision cylinder length=0.1 radius=0.025; visual cylinder length=0.1 radius=0.025
- link right_wheel: geometry collision cylinder length=0.1 radius=0.025; visual cylinder length=0.1 radius=0.025
